Commit message: Workflow optmization

File: ur5_description/urdf/ur5.urdf (robot description, URDF)
Before this commit: robot ur57_arm, 12 links, 11 joints
Joints:
- joint shoulder_pan_joint: origin xyz=0 0.13585 0 rpy=0 -1.57079632679 -1.57079632679 -> xyz=0 0.13585 0 rpy=0 0 -1.57079632679

Commit message: arm fix

File: ur5_description/urdf/ur5.urdf (robot description, URDF)
Before this commit: robot ur57_arm, 12 links, 11 joints
Joints:
- joint shoulder_pan_joint: origin xyz=0 0.13585 0 rpy=0 0 -1.57079632679 -> xyz=0 0.13585 0 rpy=0 -1.57079632679 -1.57079632679
